File: board/board.kicad_sch (KiCad schematic)
At the start: 1 part

Commit message: initial
Parts:
- removed LOGO1: Logo_Open_Hardware_Small, Symbol:OSHW-Symbol_6.7x6mm_SilkScreen, symbol Graphic:Logo_Open_Hardware_Small
- added J1: 009_1000BASE-T, on_edge:on_edge_2x05_device, symbol put_on_edge:009_1000BASE-T
Connections:
- new net magnetics/RX+: J1.4 (TD2+)
- new net magnetics/RX-: J1.5 (TD2-)
- new net magnetics/TX+: J1.2 (TD1+)
- new net magnetics/TX-: J1.3 (TD1-)
- no-connect marks 0 -> 6
Other:
- removed sheet implementation
- added sheet magnetics (magnetics.kicad_sch)
- note removed: "Input connectors go here"
- note removed: "Output connectors go here"
Changed lines of the file:
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@@
 (kicad_sch (version 20211123) (generator eeschema)
   (paper "A4")
-  (text "Output connectors go here" (at 224.79 88.9 0)
-    (effects (font (size 1.27 1.27)) (justify left bottom))
+  (no_connect (at 101.6 102.87))
+  (no_connect (at 88.9 110.49))
+  (no_connect (at 91.44 110.49))
+  (no_connect (at 101.6 100.33))
+  (no_connect (at 101.6 105.41))
+  (no_connect (at 101.6 97.79))
+  (wire (pts (xy 101.6 92.71) (xy 116.84 92.71))
+    (stroke (width 0) (type default) (color 0 0 0 0))
   )
-  (text "Input connectors go here" (at 49.53 88.9 0)
-    (effects (font (size 1.27 1.27)) (justify left bottom))
+  (wire (pts (xy 101.6 87.63) (xy 116.84 87.63))
+    (stroke (width 0) (type default) (color 0 0 0 0))
   )
-  (symbol (lib_id "Graphic:Logo_Open_Hardware_Small") (at 273.05 157.48 0) (unit 1)
+  (wire (pts (xy 101.6 90.17) (xy 116.84 90.17))
+    (stroke (width 0) (type default) (color 0 0 0 0))
+  )
+  (wire (pts (xy 101.6 95.25) (xy 116.84 95.25))
+    (stroke (width 0) (type default) (color 0 0 0 0))
+  )
+  (symbol (lib_id "put_on_edge:009_1000BASE-T") (at 90.17 96.52 0) (mirror y) (unit 1)
     (in_bom yes) (on_board yes) (fields_autoplaced)
-    (property "Reference" "LOGO1" (id 0) (at 273.05 150.495 0)
+    (property "Reference" "J1" (id 0) (at 90.805 78.74 0))
+    (property "Value" "009_1000BASE-T" (id 1) (at 90.805 81.28 0))
+    (property "Footprint" "on_edge:on_edge_2x05_device" (id 2) (at 82.55 80.01 0)
       (effects (font (size 1.27 1.27)) hide)
     )
-    (property "Value" "Logo_Open_Hardware_Small" (id 1) (at 273.05 163.195 0)
+    (property "Datasheet" "" (id 3) (at 82.55 80.01 0)
       (effects (font (size 1.27 1.27)) hide)
     )
-    (property "Footprint" "Symbol:OSHW-Symbol_6.7x6mm_SilkScreen" (id 2) (at 273.05 157.48 0)
-      (effects (font (size 1.27 1.27)) hide)
-    )
-    (property "Datasheet" "~" (id 3) (at 273.05 157.48 0)
-      (effects (font (size 1.27 1.27)) hide)
-    )
+    (pin "1")
+    (pin "10")
+    (pin "2")
+    (pin "3")
+    (pin "4")
+    (pin "5")
+    (pin "6")
+    (pin "7")
+    (pin "8")
+    (pin "9")
   )
-  (sheet (at 114.3 72.39) (size 60.96 62.23) (fields_autoplaced)
+  (sheet (at 116.84 82.55) (size 26.67 24.13) (fields_autoplaced)
     (stroke (width 0.1524) (type solid) (color 0 0 0 0))
     (fill (color 0 0 0 0.0000))
-    (property "Sheet name" "implementation" (id 0) (at 114.3 71.6784 0)
+    (property "Sheet name" "magnetics" (id 0) (at 116.84 81.8384 0)
       (effects (font (size 1.27 1.27)) (justify left bottom))
     )
-    (property "Sheet file" "implementation.kicad_sch" (id 1) (at 114.3 135.2046 0)
+    (property "Sheet file" "magnetics.kicad_sch" (id 1) (at 116.84 107.2646 0)
       (effects (font (size 1.27 1.27)) (justify left top))
+    )
+    (pin "TX-" input (at 116.84 90.17 180)
+      (effects (font (size 1.27 1.27)) (justify left))
+    )
+    (pin "RX-" input (at 116.84 95.25 180)
+      (effects (font (size 1.27 1.27)) (justify left))
+    )
+    (pin "RX+" input (at 116.84 92.71 180)
+      (effects (font (size 1.27 1.27)) (justify left))
+    )
+    (pin "TX+" input (at 116.84 87.63 180)
+      (effects (font (size 1.27 1.27)) (justify left))
     )
   )
   (sheet_instances
     (path "/" (page "1"))
-    (path "/767ce4c6-0e55-4543-92f0-34cb8237a544" (page "2"))
+    (path "/8fbd7889-9183-4cb7-8226-dfa49ef07f6c" (page "2"))
   )
   (symbol_instances
-    (path "/b72b6f4a-7489-40f2-bb90-d75ae01aa368"
-      (reference "LOGO1") (unit 1) (value "Logo_Open_Hardware_Small") (footprint "Symbol:OSHW-Symbol_6.7x6mm_SilkScreen")
+    (path "/93b280f7-6a72-461f-a036-cc0699ef1814"
+      (reference "J1") (unit 1) (value "009_1000BASE-T") (footprint "on_edge:on_edge_2x05_device")
+    )
+    (path "/8fbd7889-9183-4cb7-8226-dfa49ef07f6c/20bf1f96-1d2d-426a-a3b2-eab2fb9f6545"
+      (reference "J2") (unit 1) (value "M12D-04PFFP-SF8001") (footprint "b095:M12D")
     )
   )
